File: kimchi_ulid.sch (KiCad schematic (older format))
At the start: 8 parts, among them J1 DF40HC(3.5)-60DS, J2 DF40HC(3.5)-60DS, U1 24C32

Commit message: Mockup Progress
Added standard SMT tactile switches to represent the button pad layout for both D-Pad and Face Buttons. Added dummy Analog Sticks for mockup purposes until we can get samples of the Nintendo Switch Joy Con replacement sticks. Also added USB port and Audio Codec/Headset jack, currently working through codec shecmatic implemenation.
Parts:
- added J3: KUSBX-AS1N-B, kimchi_ulid:USB_A, symbol kimchi_ulid:KUSBX-AS1N-B
- added J4: 54-00176, kimchi_ulid:54-00176, symbol kimchi_ulid:54-00176
- added J5: SGTL5000XNLA3, kimchi_ulid:QFN40P300X300X60-21N, symbol kimchi_ulid:SGTL5000XNLA3
- added JS1, JS2: Keyes_HW-504, kimchi_ulid:Keyes_JoyStick, symbol kimchi_ulid:Keyes_HW-504
- added SW1, SW2, SW3, SW4, SW5, SW6, SW7, SW8: TL3301NF260QG, kimchi_ulid:TL3301NF260QG, symbol kimchi_ulid:TL3301NF260QG
- H1, H2, H3, H4: symbol Mechanical:MountingHole_Pad -> kimchi_ulid-rescue:MountingHole_Pad-Mechanical
- LOGO1: symbol Graphic:Logo_Open_Hardware_Small -> kimchi_ulid-rescue:Logo_Open_Hardware_Small-Graphic
Connections:
- net GND: now also J3.4 (GND), J3.5 (Shield), J4.1
- net USB2_DN: now also J3.2 (D-)
- net USB2_DP: now also J3.3 (D+)
- net USB2_VBUS: now also J3.1 (VBUS)
- new net HPOUT_L: J4.2, J5.1 (HP_R)
- new net HPOUT_R: J4.3, J5.4 (HP_L)
- new net MIC_BIAS: J5.11 (MIC_BIAS)
- new net MIC_IN: J4.4, J5.10 (MIC)
